File: Light_bicycle/Hareware/light_bicycle/light_bicycle.kicad_pcb (KiCad board)
At the start: 2 copper layers, 79 parts, among them J1 USART1, J2 电池, J3 SWD, J4 SWD, J5 USB_C_Receptacle, SW1 SMD_4.2x3.2mm_h2.5mm, SW2 SMD_4.2x3.2mm_h2.5mm, SW3 SMD_4.2x3.2mm_h2.5mm, U4 TP4056-42-ESOP8, Y1 8MHz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

Commit message: RTT 调试
Parts:
- moved C32 13.9 mm to (159.4, 25.3)
- moved C33 13.9 mm to (159.4, 28.3)
- moved C34 13.9 mm to (163.6, 25.1)
- moved U5 13.9 mm to (147.7, 19.8)
Changed lines of the file:
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@@
 	(footprint "SparkFun-Capacitor:C_0603_1608Metric"
 		(layer "F.Cu")
-		(at 177.435736 25.395736)
+		(at 163.585736 25.079736)
 		(tags "SparkFun capacitor")
 		(property "Reference" "C34"
@@
 	(footprint "SparkFun-Capacitor:C_0805_2012Metric"
 		(layer "F.Cu")
-		(at 173.205736 25.645736)
+		(at 159.355736 25.329736)
 		(descr "Capacitor SMD 0805 (2012 Metric), square (rectangular) end terminal, IPC_7351 nominal, (Body size source: IPC-SM-782 page 76, https://www.pcb-3d.com/wordpress/wp-content/uploads/ipc-sm-782a_amendment_1_and_2.pdf, https://docs.google.com/spreadsheets/d/1BsfQQcO9C6DZCsRaXUlFlo91Tg2WpOkGARC1WS5S8t0/edit?usp=sharing), generated with kicad-footprint-generator")
 		(tags "SparkFun capacitor")
@@
 	(footprint "BrookDawn_Library:MPU6500"
 		(layer "F.Cu")
-		(at 161.54 20.148)
+		(at 147.69 19.832)
 		(property "Reference" "U5"
 			(at 0 -0.5 0)
@@
 	(footprint "SparkFun-Capacitor:C_0805_2012Metric"
 		(layer "F.Cu")
-		(at 173.205736 28.655736)
+		(at 159.355736 28.339736)
 		(descr "Capacitor SMD 0805 (2012 Metric), square (rectangular) end terminal, IPC_7351 nominal, (Body size source: IPC-SM-782 page 76, https://www.pcb-3d.com/wordpress/wp-content/uploads/ipc-sm-782a_amendment_1_and_2.pdf, https://docs.google.com/spreadsheets/d/1BsfQQcO9C6DZCsRaXUlFlo91Tg2WpOkGARC1WS5S8t0/edit?usp=sharing), generated with kicad-footprint-generator")
 		(tags "SparkFun capacitor")
