File: BLDC/ProPrj_BLDCcontroller_2025-09-27/ProPrj_BLDCcontroller_2025-09-27.kicad_sch (KiCad schematic)
At the start: 54 parts, among them CN1 WAFER-GH1.25-7PLB, J1 Conn_01x01, J2 Conn_01x01, J3 Conn_01x01, J4 Conn_01x01, J5 Conn_01x01, SW2 SMD_4.2x3.2mm_h2.5mm, U1 SGM2019-3.3YN5G/TR, U10 AS5600-ASOM, U2 TPS54302DDCR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

Commit message: BLDC 更新
Parts:
- removed 251, 2511: ~, ProPrj_BLD-easyedapro:, symbol ProPrj_BLD-easyedapro:Short-Symbol
- added R7: 0, SparkFun-Resistor:R_0603_1608Metric, symbol SparkFun-Resistor:0_0603
- C19: footprint ProPrj_BLD-easyedapro:C0603 -> Capacitor_SMD:C_0603_1608Metric
- C22: value 100nF -> 1uF
Connections:
- net OUT3 is gone; now on net MOTOR3: U5.9 (OUT3)
- net SCL is gone; now on net PB6: R10.2, U10.7 (SCL)
- net SDA is gone; now on net PB7: R11.1, U10.6 (SDA)
- net VDD is gone; now on net 3.3V: U3.1 (VDD), U3.24 (VDD), U3.48 (VDD), U3.9 (VDDA)
- net VSS is gone; now on net GND: U3.23 (VSS), U3.47 (VSS), U3.8 (VSSA)
- net GND: now also C22.1, C23.1, J2.1 (Pin_1), U10.4 (GND), Y1.2, Y1.4, R7.1; no longer C21.2, U5.19 (COMPO#)
- net PA6: now also U5.26 (EN1)
- net PA7: now also U5.24 (EN2)
- net PB0: now also U5.22 (EN3)
- net PGND: now also R7.2; no longer J2.1 (Pin_1)
- new net: C21.2, U5.19 (COMPO#)
